File: AmigaUSBMouseV2.brd (EAGLE design)
At the start: 32.5 x 30.7 mm, 5 parts

Commit message: PDFs and layout fixes
Parts:
- added PWR_BRIDGE: (no value), pinhead:1X02
- AMIGA, PWR: value 0 -> (none)
- moved L 3.81 mm to (9.93, 9.60)
- moved R 1.02 mm to (10.5, 23.6), turned to 0 degrees
Connections:
- net GND: now also PWR_BRIDGE.1
- net RAW: now also PWR_BRIDGE.2
Routing:
- net RAW: track 7.08 -> 33.3 mm
- net GND: track 78.8 -> 69.6 mm
- net BTN_L: track 8.71 -> 6.77 mm
- net MOUSE_RIGHT: track 28.0 -> 27.1 mm
- net MOUSE_LEFT: track 9.15 -> 8.32 mm
